File: 2023-2024 Main Board/Motherboard23-24/5VProtection.kicad_sch (KiCad schematic)
At the start: 0 parts

Commit message: Added Schematic for Steering and Throttle
Parts:
- added D6: DIODE, Diode_THT:D_DO-15_P5.08mm_Vertical_KathodeUp, symbol Motherboard_2023-rescue:DIODE-pspice
- added D7: D_Zener, Diode_THT:D_DO-15_P5.08mm_Vertical_KathodeUp, symbol Device:D_Zener
- added J7: Conn_01x02_Male, TerminalBlock_Phoenix:TerminalBlock_Phoenix_MKDS-1,5-2-5.08_1x02_P5.08mm_Horizontal, symbol Motherboard_2023-rescue:Conn_01x02_Male-Connector
- added TH1: Thermistor, Resistor_THT:R_Axial_DIN0414_L11.9mm_D4.5mm_P5.08mm_Vertical, symbol Device:Thermistor
Connections:
- new net: D6.1 (K), J7.1 (Pin_1)
- new net: D6.2 (A), TH1.2
- new net +5V: D7.1 (K), TH1.1
- new net GND: D7.2 (A), J7.2 (Pin_2)
Other:
- note added: "5V Regulator In"
- note added: "Common Ground"
Changed lines of the file:
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@@
 (kicad_sch (version 20230121) (generator eeschema)
   (paper "A4")
+  (junction (at 121.92 76.2) (diameter 0) (color 0 0 0 0)
+  )
+  (junction (at 92.71 101.6) (diameter 0) (color 0 0 0 0)
+  )
+  (wire (pts (xy 95.25 76.2) (xy 106.68 76.2))
+    (stroke (width 0) (type default))
+  )
+  (wire (pts (xy 85.09 77.47) (xy 85.09 76.2))
+    (stroke (width 0) (type default))
+  )
+  (wire (pts (xy 121.92 101.6) (xy 121.92 91.44))
+    (stroke (width 0) (type default))
+  )
+  (wire (pts (xy 116.84 76.2) (xy 121.92 76.2))
+    (stroke (width 0) (type default))
+  )
+  (wire (pts (xy 64.77 80.01) (xy 64.77 101.6))
+    (stroke (width 0) (type default))
+  )
+  (wire (pts (xy 92.71 101.6) (xy 121.92 101.6))
+    (stroke (width 0) (type default))
+  )
+  (wire (pts (xy 121.92 76.2) (xy 156.21 76.2))
+    (stroke (width 0) (type default))
+  )
+  (wire (pts (xy 64.77 77.47) (xy 85.09 77.47))
+    (stroke (width 0) (type default))
+  )
+  (wire (pts (xy 64.77 101.6) (xy 92.71 101.6))
+    (stroke (width 0) (type default))
+  )
+  (wire (pts (xy 121.92 76.2) (xy 121.92 83.82))
+    (stroke (width 0) (type default))
+  )
+  (text "Common Ground" (at 41.91 81.28 0)
+    (effects (font (size 1.27 1.27)) (justify left bottom))
+  )
+  (text "5V Regulator In\n" (at 41.91 78.74 0)
+    (effects (font (size 1.27 1.27)) (justify left bottom))
+  )
+  (symbol (lib_id "Device:D_Zener") (at 121.92 87.63 270) (unit 1)
+    (in_bom yes) (on_board yes) (dnp no)
+    (property "Reference" "D7" (at 123.952 86.4616 90)
+      (effects (font (size 1.27 1.27)) (justify left))
+    )
+    (property "Value" "D_Zener" (at 123.952 88.773 90)
+      (effects (font (size 1.27 1.27)) (justify left))
+    )
+    (property "Footprint" "Diode_THT:D_DO-15_P5.08mm_Vertical_KathodeUp" (at 121.92 87.63 0)
+      (effects (font (size 1.27 1.27)) hide)
+    )
+    (property "Datasheet" "~" (at 121.92 87.63 0)
+      (effects (font (size 1.27 1.27)) hide)
+    )
+    (pin "1")
+    (pin "2")
+    (instances
+      (project "Motherboard23-24"
+        (path "/418d1727-08ff-41e8-954f-e6e13e4fb4ca/7d37a3b4-ae31-4786-acc0-9fb13a05600d"
+          (reference "D7") (unit 1)
+        )
+      )
+      (project "Motherboard_2023"
+        (path "/a08b3282-09d4-42be-9393-f12c9a3e8b21/00000000-0000-0000-0000-000063cda050"
+          (reference "D2") (unit 1)
+        )
+      )
+    )
+  )
+  (symbol (lib_id "Motherboard_2023-rescue:Conn_01x02_Male-Connector") (at 59.69 77.47 0) (unit 1)
+    (in_bom yes) (on_board yes) (dnp no)
+    (property "Reference" "J7" (at 62.4332 72.8726 0)
+      (effects (font (size 1.27 1.27)))
+    )
+    (property "Value" "Conn_01x02_Male" (at 62.4332 75.184 0)
+      (effects (font (size 1.27 1.27)))
+    )
+    (property "Footprint" "TerminalBlock_Phoenix:TerminalBlock_Phoenix_MKDS-1,5-2-5.08_1x02_P5.08mm_Horizontal" (at 59.69 77.47 0)
+      (effects (font (size 1.27 1.27)) hide)
+    )
+    (property "Datasheet" "~" (at 59.69 77.47 0)
+      (effects (font (size 1.27 1.27)) hide)
+    )
+    (pin "1")
+    (pin "2")
+    (instances
+      (project "Motherboard23-24"
+        (path "/418d1727-08ff-41e8-954f-e6e13e4fb4ca/7d37a3b4-ae31-4786-acc0-9fb13a05600d"
+          (reference "J7") (unit 1)
+        )
+      )
+      (project "Motherboard_2023"
+        (path "/a08b3282-09d4-42be-9393-f12c9a3e8b21"
+          (reference "J7") (unit 1)
+        )
+        (path "/a08b3282-09d4-42be-9393-f12c9a3e8b21/00000000-0000-0000-0000-000063cda050"
+          (reference "J7") (unit 1)
+        )
+      )
+    )
+  )
+  (symbol (lib_id "Motherboard_2023-rescue:DIODE-pspice") (at 90.17 76.2 0) (unit 1)
+    (in_bom yes) (on_board yes) (dnp no)
+    (property "Reference" "D6" (at 90.17 69.469 0)
+      (effects (font (size 1.27 1.27)))
+    )
+    (property "Value" "DIODE" (at 90.17 71.7804 0)
+      (effects (font (size 1.27 1.27)))
+    )
+    (property "Footprint" "Diode_THT:D_DO-15_P5.08mm_Vertical_KathodeUp" (at 90.17 76.2 0)
+      (effects (font (size 1.27 1.27)) hide)
+    )
+    (property "Datasheet" "~" (at 90.17 76.2 0)
+      (effects (font (size 1.27 1.27)) hide)
+    )
+    (pin "1")
+    (pin "2")
+    (instances
+      (project "Motherboard23-24"
+        (path "/418d1727-08ff-41e8-954f-e6e13e4fb4ca/7d37a3b4-ae31-4786-acc0-9fb13a05600d"
+          (reference "D6") (unit 1)
+        )
+      )
+      (project "Motherboard_2023"
+        (path "/a08b3282-09d4-42be-9393-f12c9a3e8b21/00000000-0000-0000-0000-000063cda050"
+          (reference "D1") (unit 1)
+        )
+      )
+    )
+  )
+  (symbol (lib_id "Device:Thermistor") (at 111.76 76.2 270) (unit 1)
+    (in_bom yes) (on_board yes) (dnp no)
+    (property "Reference" "TH1" (at 111.76 70.0532 90)
+      (effects (font (size 1.27 1.27)))
+    )
+    (property "Value" "Thermistor" (at 111.76 72.3646 90)
+      (effects (font (size 1.27 1.27)))
+    )
+    (property "Footprint" "Resistor_THT:R_Axial_DIN0414_L11.9mm_D4.5mm_P5.08mm_Vertical" (at 111.76 76.2 0)
+      (effects (font (size 1.27 1.27)) hide)
+    )
+    (property "Datasheet" "~" (at 111.76 76.2 0)
+      (effects (font (size 1.27 1.27)) hide)
+    )
+    (pin "1")
+    (pin "2")
+    (instances
+      (project "Motherboard23-24"
+        (path "/418d1727-08ff-41e8-954f-e6e13e4fb4ca/7d37a3b4-ae31-4786-acc0-9fb13a05600d"
+          (reference "TH1") (unit 1)
+        )
+      )
+      (project "Motherboard_2023"
+        (path "/a08b3282-09d4-42be-9393-f12c9a3e8b21/00000000-0000-0000-0000-000063cda050"
+          (reference "TH1") (unit 1)
+        )
+      )
+    )
+  )
+  (symbol (lib_id "power:GND") (at 92.71 101.6 0) (unit 1)
+    (in_bom yes) (on_board yes) (dnp no)
+    (property "Reference" "#PWR01" (at 92.71 107.95 0)
+      (effects (font (size 1.27 1.27)) hide)
+    )
+    (property "Value" "GND" (at 92.837 105.9942 0)
+      (effects (font (size 1.27 1.27)))
+    )
+    (property "Footprint" "" (at 92.71 101.6 0)
+      (effects (font (size 1.27 1.27)) hide)
+    )
+    (property "Datasheet" "" (at 92.71 101.6 0)
+      (effects (font (size 1.27 1.27)) hide)
+    )
+    (pin "1")
+    (instances
+      (project "Motherboard23-24"
+        (path "/418d1727-08ff-41e8-954f-e6e13e4fb4ca/7d37a3b4-ae31-4786-acc0-9fb13a05600d"
+          (reference "#PWR01") (unit 1)
+        )
+      )
+      (project "Motherboard_2023"
+        (path "/a08b3282-09d4-42be-9393-f12c9a3e8b21/00000000-0000-0000-0000-000063cda050"
+          (reference "#PWR026") (unit 1)
+        )
+      )
+    )
+  )
+  (symbol (lib_id "power:+5V") (at 156.21 76.2 0) (unit 1)
+    (in_bom yes) (on_board yes) (dnp no)
+    (property "Reference" "#PWR02" (at 156.21 80.01 0)
+      (effects (font (size 1.27 1.27)) hide)
+    )
+    (property "Value" "+5V" (at 156.591 71.8058 0)
+      (effects (font (size 1.27 1.27)))
+    )
+    (property "Footprint" "" (at 156.21 76.2 0)
+      (effects (font (size 1.27 1.27)) hide)
+    )
+    (property "Datasheet" "" (at 156.21 76.2 0)
+      (effects (font (size 1.27 1.27)) hide)
+    )
+    (pin "1")
+    (instances
+      (project "Motherboard23-24"
+        (path "/418d1727-08ff-41e8-954f-e6e13e4fb4ca/7d37a3b4-ae31-4786-acc0-9fb13a05600d"
+          (reference "#PWR02") (unit 1)
+        )
+      )
+      (project "Motherboard_2023"
+        (path "/a08b3282-09d4-42be-9393-f12c9a3e8b21/00000000-0000-0000-0000-000063cda050"
+          (reference "#PWR027") (unit 1)
+        )
+      )
+    )
+  )
 )
