File: 2023-2024 Main Board/Motherboard23-24/safety.kicad_sch (KiCad schematic)
At the start: 0 parts

Commit message: Added Schematic for Steering and Throttle
Parts:
- added C1, C2, C3: 0.1µF, Capacitor_THT:CP_Radial_D5.0mm_P2.50mm, symbol Device:C
- added J10: Conn_01x04_Male, TerminalBlock_Phoenix:TerminalBlock_Phoenix_MKDS-3-4-5.08_1x04_P5.08mm_Horizontal, symbol Motherboard_2023-rescue:Conn_01x04_Male-Connector
- added J4: Conn_01x03_Male, TerminalBlock_Phoenix:TerminalBlock_Phoenix_MKDS-3-3-5.08_1x03_P5.08mm_Horizontal, symbol Motherboard_2023-rescue:Conn_01x03_Male-Connector
- added Q1: Q_NMOS_GDS, Connector_PinHeader_2.54mm:PinHeader_1x03_P2.54mm_Vertical, symbol Device:Q_NMOS_GDS
- added R10, R11, R19, R20, R21, R22, R23, R24, R28, R6, R7, R8, R9: 1k, Resistor_THT:R_Axial_DIN0207_L6.3mm_D2.5mm_P10.16mm_Horizontal, symbol Device:R
- added R12, R13, R14, R15, R16, R17, R18, R26, R27: 10k, Resistor_THT:R_Axial_DIN0207_L6.3mm_D2.5mm_P10.16mm_Horizontal, symbol Device:R
- added R25: 330, Resistor_THT:R_Axial_DIN0207_L6.3mm_D2.5mm_P10.16mm_Horizontal, symbol Device:R
- added R29: 100k, Resistor_THT:R_Axial_DIN0207_L6.3mm_D2.5mm_P10.16mm_Horizontal, symbol Device:R
- added U3: CD4081BE, CD4081BE (AND):DIP794W45P254L1969H508Q14, symbol CD4081BE:CD4081BE
- added U4: CD4069UBE, CD4069UBE (Inverter):DIP794W45P254L1969H508Q14, symbol CD4069UBE:CD4069UBE
Connections:
- new net: R18.1, U3.13 (H)
- new net: R27.2, U3.11 (M=G.M)
- new net: R25.1, U3.3 (J=A.B)
- new net: Q1.1 (G), R25.2, R29.1
- new net: R22.2, U4.11 (E)
- new net: R23.1, U4.13 (F)
- new net: R28.1, U4.2 (~{A})
- new net: R19.1, U4.3 (B)
- new net: R20.2, U4.5 (C)
- new net: R21.1, U4.9 (D)
- new net: R24.1, U3.4 (K=C.D)
- new net: R24.2, U3.2 (B)
- new net: R17.1, U3.12 (G)
- new net: R26.2, U3.10 (L=E.F)
- new net: R15.1, U3.8 (E)
- new net: R16.1, U3.9 (F)
- new net +12V: J10.2 (Pin_2), R19.2, R20.1, R21.2, R22.1, R23.2, U3.14 (VDD), U4.14 (VDD)
- new net Brake: C2.1, J4.2 (Pin_2), R10.2, R7.1
- new net Brake_Output: R10.1, R13.1, U3.6 (D)
- new net GND: C1.2, C2.2, C3.2, J10.3 (Pin_3), J10.4 (Pin_4), Q1.3 (S), R12.2, R13.2, R14.2, R15.2, R16.2, R17.2, R18.2, R26.1, R27.1, R29.2, R6.2, R7.2, R8.2, U3.7 (VSS), U4.10 (~{E}), U4.12 (~{F}), U4.4 (~{B}), U4.6 (~{C}), U4.7 (VSS), U4.8 (~{D})
- new net Neutral: C1.1, J4.1 (Pin_1), R6.1, R9.2
- new net Neutral_Inverted: R28.2, U3.1 (A)
- new net Neutral_Output: R12.1, R9.1, U4.1 (A)
- new net Safety_Signal: J10.1 (Pin_1), Q1.2 (D)
- new net Seat: C3.1, J4.3 (Pin_3), R11.2, R8.1
- new net Seat_Output: R11.1, R14.1, U3.5 (C)
Other:
- note added: "AND Logic"
- note added: "Inverter Logic"
- note added: "Sensor Filtering"
- note added: "System Inputs"
