File: 2023-2024 Main Board/Motherboard23-24/safetystart.kicad_sch (KiCad schematic)
At the start: 9 parts, among them J11 Conn_01x06_Male, J12 VCF4-1000, J13 VCF4-1000, J14 Conn_01x03_Male, J15 VCF4-1000, J16 VCF4-1000, J17 Conn_01x02_Male, Q2 Q_NMOS_GDS

Commit message: first draft of 23-24 Main Board
Parts:
- J11: footprint TerminalBlock_Phoenix:TerminalBlock_Phoenix_MKDS-3-6-5.08_1x06_P5.08mm_Horizontal -> TerminalBlock_Phoenix:TerminalBlock_Phoenix_MKDS-1,5-6-5.08_1x06_P5.08mm_Horizontal
Connections:
- no-connect marks 0 -> 1
Changed lines of the file:
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@@
   (junction (at 171.45 58.42) (diameter 0) (color 0 0 0 0)
   )
+  (no_connect (at 138.43 68.58))
   (wire (pts (xy 219.71 45.72) (xy 212.09 45.72))
     (stroke (width 0) (type default))
@@
     (stroke (width 0) (type default))
   )
-  (wire (pts (xy 143.51 43.18) (xy 143.51 50.8))
+  (wire (pts (xy 143.51 43.18) (xy 143.51 53.34))
     (stroke (width 0) (type default))
   )
@@
     (stroke (width 0) (type default))
   )
-  (wire (pts (xy 173.99 50.8) (xy 143.51 50.8))
+  (wire (pts (xy 173.99 53.34) (xy 143.51 53.34))
     (stroke (width 0) (type default))
   )
@@
     (stroke (width 0) (type default))
   )
-  (wire (pts (xy 173.99 68.58) (xy 173.99 50.8))
+  (wire (pts (xy 173.99 68.58) (xy 173.99 53.34))
     (stroke (width 0) (type default))
   )
@@
     (effects (font (size 1.4986 1.4986) (thickness 0.2997) bold) (justify left bottom))
   )
-  (text "Fuel Solenoid" (at 139.7 48.26 90)
-    (effects (font (size 0.508 0.508) (thickness 0.1016) bold) (justify left bottom))
-  )
-  (text "Start Button \n" (at 205.74 43.18 0)
+  (text "Fuel Solenoid" (at 148.59 53.34 0)
+    (effects (font (size 0.508 0.508) (thickness 0.1016) bold) (justify right bottom))
+  )
+  (text "Start Button \n" (at 204.47 44.45 0)
     (effects (font (size 0.508 0.508) (thickness 0.1016) bold) (justify left bottom))
   )
@@
     (effects (font (size 1.4986 1.4986) (thickness 0.2997) bold) (justify left bottom))
   )
-  (text "Spark\n" (at 137.16 46.99 90)
-    (effects (font (size 0.508 0.508) (thickness 0.1016) bold) (justify left bottom))
+  (text "Spark\n" (at 140.97 52.07 0)
+    (effects (font (size 0.508 0.508) (thickness 0.1016) bold) (justify right bottom))
   )
   (label "Comp_Switch" (at 97.79 48.26 0) (fields_autoplaced)
@@
       (effects (font (size 1.27 1.27)) (justify right))
     )
-    (property "Footprint" "TerminalBlock_Phoenix:TerminalBlock_Phoenix_MKDS-3-6-5.08_1x06_P5.08mm_Horizontal" (at 87.63 38.1 0)
-      (effects (font (size 1.27 1.27)) hide)
-    )
+    (property "Footprint" "TerminalBlock_Phoenix:TerminalBlock_Phoenix_MKDS-1,5-6-5.08_1x06_P5.08mm_Horizontal" (at 87.63 38.1 0)
+      (effects (font (size 1.27 1.27)) hide)
+    )
