File: 2023-2024 Main Board/Motherboard23-24/throttle.kicad_sch (KiCad schematic)
At the start: 0 parts

Commit message: Added Schematic for Steering and Throttle
Parts:
- added J1: Conn_01x06_Pin, symbol Connector:Conn_01x06_Pin
- added J21: Conn_01x02_Male, TerminalBlock_Phoenix:TerminalBlock_Phoenix_MKDS-1,5-2-5.08_1x02_P5.08mm_Horizontal, symbol Motherboard_2023-rescue:Conn_01x02_Male-Connector
- added J8: Conn_01x08_Male, TerminalBlock_Phoenix:TerminalBlock_Phoenix_MKDS-1,5-8-5.08_1x08_P5.08mm_Horizontal, symbol Motherboard_2023-rescue:Conn_01x08_Male-Connector
- added R31, R32, R33: R, symbol Device:R
- added U1: ARDUINO_PRO_MINI, ARDUINO_PRO_MINI:MODULE_ARDUINO_PRO_MINI, symbol ARDUINO_PRO_MINI:ARDUINO_PRO_MINI
Connections:
- new net: J1.1 (Pin_1), U1.JP1_1 (DTR)
- new net: J1.2 (Pin_2), U1.JP1_2 (TXO)
- new net: J1.3 (Pin_3), U1.JP1_3 (RXI)
- new net: J1.5 (Pin_5), J1.6 (Pin_6), U1.JP1_5 (GND), U1.JP1_6 (GND)
- new net: J8.6 (Pin_6), R31.1, U1.JP7_8 (D2)
- new net: J8.3 (Pin_3), U1.JP6_8 (A0)
- new net: J8.4 (Pin_4), U1.JP6_7 (A1)
- new net: J8.7 (Pin_7), R32.1, U1.JP7_7 (D3)
- new net: J8.8 (Pin_8), R33.1, U1.JP7_6 (D4)
- new net +5V: J8.1 (Pin_1), U1.JP6_4 (VCC_1)
- new net GND: J8.2 (Pin_2), J8.5 (Pin_5), R31.2, R32.2, R33.2, U1.JP6_2 (GND_1), U1.JP7_9 (GND_2)
- no-connect marks 0 -> 1
Other:
- note added: "Analog #1"
- note added: "Button Sig #1"
- note added: "Button Sig #2"
- note added: "DTR"
- note added: "GND"
- note added: "Joystick Deadman"
- note added: "Programming pins"
- note added: "RXI"
- note added: "TX0"

Commit message: Close to finishing up 2023-2024 Main Board Schematic
Connections:
- net GND: now also J21.2 (Pin_2)
- net at J21.1 (Pin_1): now also U1.JP7_1 (D9)
Changed lines of the file:
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@@
+    (stroke (width 0) (type default))
+  )
+  (wire (pts (xy 113.03 114.3) (xy 100.33 114.3))
     (stroke (width 0) (type default))
   )
@@
     (stroke (width 0) (type default))
   )
+  (wire (pts (xy 113.03 93.98) (xy 113.03 114.3))
+    (stroke (width 0) (type default))
+  )
   (wire (pts (xy 157.48 105.41) (xy 154.94 105.41))
     (stroke (width 0) (type default))
@@
     (stroke (width 0) (type default))
   )
+  (wire (pts (xy 175.26 63.5) (xy 175.26 93.98))
+    (stroke (width 0) (type default))
+  )
   (wire (pts (xy 100.33 83.82) (xy 123.19 83.82))
     (stroke (width 0) (type default))
@@
     (stroke (width 0) (type default))
   )
+  (wire (pts (xy 113.03 93.98) (xy 175.26 93.98))
+    (stroke (width 0) (type default))
+  )
   (wire (pts (xy 64.77 99.06) (xy 58.42 99.06))
     (stroke (width 0) (type default))
@@
   )
   (wire (pts (xy 157.48 63.5) (xy 157.48 96.52))
+    (stroke (width 0) (type default))
+  )
+  (wire (pts (xy 172.72 63.5) (xy 172.72 71.12))
     (stroke (width 0) (type default))
   )
@@
         )
       )
+    )
+  )
+  (symbol (lib_id "power:GND") (at 172.72 71.12 0) (unit 1)
+    (in_bom yes) (on_board yes) (dnp no)
+    (property "Reference" "#PWR038" (at 172.72 77.47 0)
+      (effects (font (size 1.27 1.27)) hide)
+    )
+    (property "Value" "GND" (at 172.847 74.3712 90)
+      (effects (font (size 1.27 1.27)) (justify right))
+    )
+    (property "Footprint" "" (at 172.72 71.12 0)
+      (effects (font (size 1.27 1.27)) hide)
+    )
+    (property "Datasheet" "" (at 172.72 71.12 0)
+      (effects (font (size 1.27 1.27)) hide)
+    )
+    (pin "1")
+    (instances
+      (project "Motherboard23-24"
+        (path "/418d1727-08ff-41e8-954f-e6e13e4fb4ca/1e49dcc8-e11f-4b9d-96b3-823be8a481eb"
+          (reference "#PWR038") (unit 1)
+        )
+      )
+      (project "Motherboard_2023"
+        (path "/f8df85fb-4ee1-4f8d-89fa-dcc6eddf16e2/00000000-0000-0000-0000-000063cdee43"
+          (reference "#PWR033") (unit 1)
+        )
+      )

Commit message: Added BOM
Parts:
- removed J1: Conn_01x06_Pin, symbol Connector:Conn_01x06_Pin
Connections:
- no-connect marks 1 -> 0
Other:
- note removed: "DTR"
- note removed: "GND"
- note removed: "Programming pins"
- note removed: "RXI"
- note removed: "TX0"
Changed lines of the file:
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@@
   (junction (at 162.56 101.6) (diameter 0) (color 0 0 0 0)
   )
-  (junction (at 115.57 63.5) (diameter 0) (color 0 0 0 0)
-  )
-  (no_connect (at 120.65 63.5))
   (wire (pts (xy 165.1 118.11) (xy 160.02 118.11))
     (stroke (width 0) (type default))
@@
     (stroke (width 0) (type default))
   )
-  (wire (pts (xy 123.19 63.5) (xy 123.19 83.82))
-    (stroke (width 0) (type default))
-  )
   (wire (pts (xy 154.94 115.57) (xy 154.94 118.11))
     (stroke (width 0) (type default))
@@
   )
   (wire (pts (xy 175.26 63.5) (xy 175.26 93.98))
-    (stroke (width 0) (type default))
-  )
-  (wire (pts (xy 100.33 83.82) (xy 123.19 83.82))
-    (stroke (width 0) (type default))
-  )
-  (wire (pts (xy 115.57 63.5) (xy 118.11 63.5))
-    (stroke (width 0) (type default))
-  )
-  (wire (pts (xy 115.57 63.5) (xy 115.57 119.38))
     (stroke (width 0) (type default))
   )
@@
     (stroke (width 0) (type default))
   )
-  (wire (pts (xy 100.33 78.74) (xy 128.27 78.74))
-    (stroke (width 0) (type default))
-  )
   (wire (pts (xy 152.4 83.82) (xy 137.16 83.82))
     (stroke (width 0) (type default))
@@
     (stroke (width 0) (type default))
   )
-  (wire (pts (xy 100.33 81.28) (xy 125.73 81.28))
-    (stroke (width 0) (type default))
-  )
   (wire (pts (xy 55.88 96.52) (xy 64.77 96.52))
-    (stroke (width 0) (type default))
-  )
-  (wire (pts (xy 128.27 63.5) (xy 128.27 78.74))
     (stroke (width 0) (type default))
   )
@@
   )
   (wire (pts (xy 58.42 48.26) (xy 137.16 48.26))
-    (stroke (width 0) (type default))
-  )
-  (wire (pts (xy 125.73 63.5) (xy 125.73 81.28))
     (stroke (width 0) (type default))
   )
@@
     (stroke (width 0) (type default))
   )
-  (text "Programming pins " (at 113.03 58.42 0)
-    (effects (font (size 1.27 1.27)) (justify left bottom))
-  )
-  (text "GND" (at 118.11 64.77 0)
-    (effects (font (size 0.508 0.508)) (justify right bottom))
-  )
   (text "Joystick Deadman \n" (at 160.02 74.93 90)
     (effects (font (size 0.889 0.889)) (justify left bottom))
-  )
-  (text "RXI" (at 123.19 63.5 0)
-    (effects (font (size 0.508 0.508)) (justify right bottom))
   )
   (text "Button Sig #2" (at 162.56 72.39 90)
@@
   (text "Analog #1" (at 149.86 71.12 90)
     (effects (font (size 0.889 0.889)) (justify left bottom))
-  )
-  (text "TX0" (at 125.73 63.5 0)
-    (effects (font (size 0.508 0.508)) (justify right bottom))
-  )
-  (text "DTR" (at 128.27 63.5 0)
-    (effects (font (size 0.508 0.508)) (justify right bottom))
   )
   (symbol (lib_id "Motherboard_2023-rescue:Conn_01x02_Male-Connector") (at 175.26 58.42 270) (unit 1)
@@
         )
       )
-    )
-  )
-  (symbol (lib_id "Connector:Conn_01x06_Pin") (at 123.19 58.42 270) (unit 1)
-    (in_bom yes) (on_board yes) (dnp no) (fields_autoplaced)
-    (property "Reference" "J1" (at 121.92 53.34 90)
-      (effects (font (size 1.27 1.27)))
-    )
-    (property "Value" "Conn_01x06_Pin" (at 121.92 55.88 90)
-      (effects (font (size 1.27 1.27)))
-    )
-    (property "Footprint" "" (at 123.19 58.42 0)
-      (effects (font (size 1.27 1.27)) hide)
-    )
-    (property "Datasheet" "~" (at 123.19 58.42 0)
-      (effects (font (size 1.27 1.27)) hide)
-    )
-    (pin "1")
-    (pin "2")
-    (pin "3")
-    (pin "4")
-    (pin "5")
-    (pin "6")
-    (instances
-      (project "Motherboard23-24"
-        (path "/418d1727-08ff-41e8-954f-e6e13e4fb4ca/97542c42-a706-445d-a930-fc308481bbac"
-          (reference "J1") (unit 1)
-        )
-        (path "/418d1727-08ff-41e8-954f-e6e13e4fb4ca/d15f88a3-eb3a-4abd-b913-7ade9bdcdd4a"
-          (reference "J8") (unit 1)
-        )
-        (path "/418d1727-08ff-41e8-954f-e6e13e4fb4ca/1e49dcc8-e11f-4b9d-96b3-823be8a481eb"
-          (reference "J20") (unit 1)
-        )
-      )

Commit message: first draft of 23-24 Main Board
Parts:
- R31, R32, R33: value R -> 10k; footprint (none) -> Resistor_THT:R_Axial_DIN0207_L6.3mm_D2.5mm_P10.16mm_Horizontal
Changed lines of the file:
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@@
-    (stroke (width 0) (type default))
-  )
-  (wire (pts (xy 115.57 119.38) (xy 100.33 119.38))
     (stroke (width 0) (type default))
   )
@@
       (effects (font (size 1.27 1.27)) (justify left))
     )
-    (property "Value" "R" (at 149.86 113.03 0)
-      (effects (font (size 1.27 1.27)) (justify left))
-    )
-    (property "Footprint" "" (at 153.162 111.76 90)
+    (property "Value" "10k" (at 149.86 113.03 0)
+      (effects (font (size 1.27 1.27)) (justify left))
+    )
+    (property "Footprint" "Resistor_THT:R_Axial_DIN0207_L6.3mm_D2.5mm_P10.16mm_Horizontal" (at 153.162 111.76 90)
       (effects (font (size 1.27 1.27)) hide)
     )
@@
       (effects (font (size 1.27 1.27)) (justify left))
     )
-    (property "Value" "R" (at 157.48 110.49 0)
-      (effects (font (size 1.27 1.27)) (justify left))
-    )
-    (property "Footprint" "" (at 158.242 111.76 90)
+    (property "Value" "10k" (at 157.48 110.49 0)
+      (effects (font (size 1.27 1.27)) (justify left))
+    )
+    (property "Footprint" "Resistor_THT:R_Axial_DIN0207_L6.3mm_D2.5mm_P10.16mm_Horizontal" (at 158.242 111.76 90)
       (effects (font (size 1.27 1.27)) hide)
     )
@@
       (effects (font (size 1.27 1.27)) (justify left))
     )
-    (property "Value" "R" (at 167.64 113.03 0)
-      (effects (font (size 1.27 1.27)) (justify left))
-    )
-    (property "Footprint" "" (at 163.322 111.76 90)
-      (effects (font (size 1.27 1.27)) hide)
-    )
+    (property "Value" "10k" (at 167.64 113.03 0)
+      (effects (font (size 1.27 1.27)) (justify left))
+    )
+    (property "Footprint" "Resistor_THT:R_Axial_DIN0207_L6.3mm_D2.5mm_P10.16mm_Horizontal" (at 163.322 111.76 90)
+      (effects (font (size 1.27 1.27)) hide)
+    )
